Commit message: feat: progress

File: src/my_robot/urdf/my_robot.xacro (robot description, xacro)
@@ -30,4 +30,9 @@
     <axis xyz="0 1 0" rpy="0 0 0"/>
   </joint>
+  <joint name="camera_optical_joint" type="fixed">
+    <origin xyz="0 0 0" rpy="-1.5707 0 -1.5707"/>
+    <parent link="camera"/>
+    <child link="camera_link_optical"/>
+  </joint>
   <joint type="fixed" name="hokuyo_join">
     <origin xyz="0.15 0 0.1" rpy="0 0 0"/>
@@ -191,3 +196,5 @@
     </visual>
   </link>
+  <link name="camera_link_optical">
+  </link>
 </robot>
